File: hardware/caravel_pcb_v3_FTDI/caravel_pcb_v3_FTDI.kicad_sch (KiCad schematic)
At the start: 57 parts, among them J1 USB_B_Micro - 10118193-0001LF, J2 Conn_01x02_Female, J3 Conn_01x02_Female, J4 Conn_01x14_Female, J5 Conn_01x02_Male, J6 Conn_01x02_Male, J7 Conn_01x06_Female, J8 Conn_01x02_Male, J9 Conn_01x02_Male, SW1 SW_Push - SKQGADE010, U1 FT232H, U2 SN74LVC1G125DCKR, U3 SN74LVC1G125DCKR, U4 AZ1117CH-1.8TRG1, U5 AZ1117-3.3, U6 W25Q32FVSS, U7 caravel_breakout, X1 DSC6001_10MHZ, Y1 CSTNE12M0GH5L000R0

Commit message: Complete PCB of FTDI caravel board (V3.1)
Parts:
- removed J4: Conn_01x14_Female, Connector_PinHeader_2.54mm:PinHeader_1x14_P2.54mm_Vertical, symbol Connector:Conn_01x14_Female
- removed U7: caravel_breakout, Caravel_Baord:caravel_breakout, symbol Caravel_board:caravel_breakout
- added J10: Conn_01x27_Female, Connector_PinHeader_2.54mm:PinHeader_1x27_P2.54mm_Vertical, symbol Connector:Conn_01x27_Female
- added J11: Conn_01x20_Female, Connector_PinHeader_2.54mm:PinHeader_1x20_P2.54mm_Vertical, symbol Connector:Conn_01x27_Female
- added T1: Logo, Caravel_Board:logo, symbol Caravel_pcb-rescue:Logo-Caravel_pcb
- added T2: Logo, Caravel_Board:ef_logo, symbol Caravel_board:Logo
- added U6: caravel_breakout, Caravel_Board:caravel_breakout_flexy, symbol Caravel_board:caravel_breakout
- J1: footprint striVe_foot_prints:FCI_10118193-0001LF -> strive_foot_prints:FCI_10118193-0001LF
- J7: footprint (none) -> Connector_PinHeader_2.54mm:PinHeader_1x06_P2.54mm_Vertical
- SW1: footprint striVe_foot_prints:SW4-SMD-5.2X5.2X1.5MM -> strive_foot_prints:SW4-SMD-5.2X5.2X1.5MM
- U1: footprint Package_QFP:LQFP-48_7x7mm_P0.5mm -> Package_DFN_QFN:QFN-48-1EP_7x7mm_P0.5mm_EP5.15x5.15mm
- U2, U3: footprint striVe_foot_prints:SOT65P210X110-5N -> strive_foot_prints:SOT65P210X110-5N
- U7: renamed from U6; footprint striVe_foot_prints:SOIC127P790X216-8N -> strive_foot_prints:SOIC127P790X216-8N
- X1: footprint striVe_foot_prints:DSC6001JE1A-010.0000 -> strive_foot_prints:DSC6001JE1A-010.0000
- Y1: footprint striVe_foot_prints:CSTNE12M0GH5L000R0 -> strive_foot_prints:CSTNE12M0GH5L000R0
Connections:
- net +1V8: now also J11.13 (Pin_13), J11.19 (Pin_19), J11.20 (Pin_20), U6.51 (vccd), U6.8 (vccd)
- net +3V3: now also J11.23 (Pin_23), J11.24 (Pin_24), J11.26 (Pin_26), U6.13 (vddio), U6.3 (vdda), U6.50 (vddio)
- net Caravel_CSB: now also U6.9 (Caravel_CSB)
- net Caravel_D0: now also U6.7 (Caravel_D0)
- net Caravel_D1: now also U6.6 (Caravel_D1)
- net Caravel_SCK: now also U6.4 (Caravel_SCK)
- net GND: now also J10.27 (Pin_27), J11.14 (Pin_14), J11.15 (Pin_15), J11.27 (Pin_27), U6.49 (GND), U6.52 (GND)
- net USB_CS1: now also J10.4 (Pin_4), U6.18 (mprj_io[3]_CSB)
- net USB_SCK_TXD: now also J10.5 (Pin_5), U6.19 (mprj_io[4]_SCK)
- net USB_SI: now also J10.2 (Pin_2), U6.16 (mprj_io[1]_SDO)
- net USB_SO_RXD: now also J10.3 (Pin_3), U6.17 (mprj_io[2]_SDI)
- net gpio: now also J11.17 (Pin_17), U6.5 (gpio)
- net mprj_io[0]: now also J10.1 (Pin_1), U6.15 (mprj_io[0])
- net mprj_io[10]: now also J10.11 (Pin_11), U6.25 (mprj_io[10])
- net mprj_io[11]: now also J10.12 (Pin_12), U6.26 (mprj_io[11])
- net mprj_io[12]: now also J10.13 (Pin_13), U6.27 (mprj_io[12])
- net mprj_io[13]: now also J10.14 (Pin_14), U6.28 (mprj_io[13])
- net mprj_io[14]: now also J10.15 (Pin_15), U6.29 (mprj_io[14])
- net mprj_io[15]: now also J10.16 (Pin_16), U6.30 (mprj_io[15])
- net mprj_io[16]: now also J10.17 (Pin_17), U6.31 (mprj_io[16])
- net mprj_io[17]: now also J10.18 (Pin_18), U6.32 (mprj_io[17])
- net mprj_io[18]: now also J10.19 (Pin_19), U6.33 (mprj_io[18])
- net mprj_io[19]: now also J10.20 (Pin_20), U6.34 (mprj_io[19])
- net mprj_io[20]: now also J10.21 (Pin_21), U6.35 (mprj_io[20])
- net mprj_io[21]: now also J10.22 (Pin_22), U6.36 (mprj_io[21])
- net mprj_io[22]: now also J10.23 (Pin_23), U6.37 (mprj_io[22])
- net mprj_io[23]: now also J10.24 (Pin_24), U6.38 (mprj_io[23])
- net mprj_io[24]: now also J10.25 (Pin_25), U6.39 (mprj_io[24])
- net mprj_io[25]: now also J10.26 (Pin_26), U6.40 (mprj_io[25])
- net mprj_io[26]: now also J11.12 (Pin_12), U6.41 (mprj_io[26])
- net mprj_io[27]: now also J11.11 (Pin_11), U6.42 (mprj_io[27])
- net mprj_io[28]: now also J11.10 (Pin_10), U6.43 (mprj_io[28])
- net mprj_io[29]: now also J11.9 (Pin_9), U6.44 (mprj_io[29])
- net mprj_io[30]: now also J11.8 (Pin_8), U6.45 (mprj_io[30])
- net mprj_io[31]: now also J11.7 (Pin_7), U6.46 (mprj_io[31])
- net mprj_io[32]: now also J11.6 (Pin_6), U6.47 (mprj_io[32])
- net mprj_io[33]: now also J11.5 (Pin_5), U6.48 (mprj_io[33])
- net mprj_io[34]: now also J11.4 (Pin_4), U6.53 (mprj_io[34])
- net mprj_io[35]: now also J11.3 (Pin_3), U6.54 (mprj_io[35])
- net mprj_io[36]: now also J11.2 (Pin_2), U6.55 (mprj_io[36])
- net mprj_io[37]: now also J11.1 (Pin_1), U6.56 (mprj_io[37])
- net mprj_io[5]_ser_rx: now also J10.6 (Pin_6), U6.20 (mprj_io[5]_ser_rx)
- net mprj_io[6]_ser_tx: now also J10.7 (Pin_7), U6.21 (mprj_io[6]_ser_tx)
- net mprj_io[7]: now also J10.8 (Pin_8), U6.22 (mprj_io[7])
- net mprj_io[8]: now also J10.9 (Pin_9), U6.23 (mprj_io[8])
- net mprj_io[9]: now also J10.10 (Pin_10), U6.24 (mprj_io[9])
- net vccd1: now also J11.21 (Pin_21), U6.1 (vccd1)
- net vccd2: now also J11.18 (Pin_18), U6.14 (vccd2)
- net vdda1: now also J11.25 (Pin_25), U6.2 (vdda1)
- net vdda2: now also J11.22 (Pin_22), U6.12 (vdda2)
- net xclk: now also J11.16 (Pin_16), U6.10 (xclk)
- net ~{RST}: now also U6.11 (~{RST})
Other:
- note added: "IO Connectors"

Commit message: update FTDI footprint
Parts:
- U1: footprint Package_DFN_QFN:QFN-48-1EP_7x7mm_P0.5mm_EP5.15x5.15mm -> Package_DFN_QFN:QFN-48-1EP_8x8mm_P0.5mm_EP6.2x6.2mm
Changed lines of the file:
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@@
     (property "Reference" "U1" (id 0) (at 68.58 115.57 0))
     (property "Value" "FT232H" (id 1) (at 73.66 115.57 0))
-    (property "Footprint" "Package_DFN_QFN:QFN-48-1EP_7x7mm_P0.5mm_EP5.15x5.15mm" (id 2) (at 85.09 151.13 0)
+    (property "Footprint" "Package_DFN_QFN:QFN-48-1EP_8x8mm_P0.5mm_EP6.2x6.2mm" (id 2) (at 85.09 151.13 0)
       (effects (font (size 1.27 1.27)) hide)
     )
@@
     )
     (path "/992b5010-a26d-41dd-b0c4-3690c286ab42"
-      (reference "U1") (unit 1) (value "FT232H") (footprint "Package_DFN_QFN:QFN-48-1EP_7x7mm_P0.5mm_EP5.15x5.15mm")
+      (reference "U1") (unit 1) (value "FT232H") (footprint "Package_DFN_QFN:QFN-48-1EP_8x8mm_P0.5mm_EP6.2x6.2mm")
     )
     (path "/2694ce6e-725b-4dc5-b62e-3db1157c7f54"
