File: hardware/development/caravel-dev-v5-M.2/Fab-Drawing-caravel-dev-v5-M.2.kicad_pcb (KiCad board)
At the start: 2 copper layers, 76.2 x 73.8 mm, 64 parts, among them J1 USB_B_Micro - 10118193-0001LF, J10 Conn_01x27_Female, J11 Conn_01x20_Female, J2 Conn_01x02_Female, J3 Conn_01x02_Male, J4 Conn_01x03_Female, J5 Conn_01x02_Male, J6 Conn_01x02_Male, J7 Conn_01x06_Female, J8 Conn_01x02_Male, J9 Conn_01x02_Male, SW1 SW_Push - SKQGADE010, T1 Logo, T2 Logo, U1 FT232H, U2 SN74LVC1G125DCKR, U3 SN74LVC1G125DCKR, U4 MCP1319MT-29LE-OT, U5 TAR5SxxU_SOT353F, U6 TAR5SxxU_SOT353F, U7 W25Q32FVSS, U8 caravel-M.2-card, X1 DSC6001_10MHZ, Y1 CSTNE12M0GH5L000R0

Commit message: add caravel REV5B Fab drawing
Parts:
- removed the D1 at (150.8, 146.9)
- removed the R3 at (144.4, 143.4)
- removed U4: MCP1319MT-29LE-OT, Caravel_Board:PoR_5_SOT23
- added C18: 0.1uF, Capacitor_SMD:C_0805_2012Metric, F.Cu at (160.0, 181.8)
- added C19: 1uF, Capacitor_SMD:C_0805_2012Metric, F.Cu at (160.0, 175.6)
- added C20: 0.01uF, Capacitor_SMD:C_0805_2012Metric, F.Cu at (128.4, 125.2)
- added C21: 0.1uF, Capacitor_SMD:C_0805_2012Metric, F.Cu at (122.7, 125.1)
- added C22: 10uF, Capacitor_SMD:C_0805_2012Metric, F.Cu at (125.5, 126.1)
- added D2: RED, LED_SMD:LED_1206_3216Metric, F.Cu at (150.9, 146.9)
- added FB1: 600R/0.5A, Inductor_SMD:L_0805_2012Metric, F.Cu at (125.5, 124.2)
- added J12: Conn_01x04_Pin, Connector_PinHeader_2.54mm:PinHeader_1x04_P2.54mm_Vertical, F.Cu at (136.9, 130.2)
- added R4: 150, Resistor_SMD:R_0805_2012Metric, F.Cu at (148.3, 152.3)
- C1: value 0.01uf - CC0805JRX7R9BB103 -> 0.01uF
- C10, C13: value 1uf - CC0805KKX5R8BB105 -> 1uF
- C11, C14: value 0.01uf - CC0805KRX7R9BB103 -> 0.01uF
- C12, C15: value 10uf - CC0805KKX5R8BB106 -> 10uF
- C16: value 0.1uf - CC0805KRX7R9BB104 -> 10uF
- C17: value 0.1uf - CC0805KRX7R9BB104 -> 0.01uF
- C2, C3, C4, C5, C6, C7, C8, C9: value 0.1uf - CC0805KRX7R9BB104 -> 0.1uF
- D1: renamed from D2; value LED - 17-215SURC/S530-A2/TR8 -> RED
- D3, D4: value LED - 17-215SURC/S530-A2/TR8 -> RED
- J1: value USB_B_Micro - 10118193-0001LF -> USB_B_Micro
- J10: value Conn_01x27_Female -> Conn_01x28_Pin
- J11: value Conn_01x20_Female -> Conn_01x28_Pin
- J2: value Conn_01x02_Female -> Conn_01x02_Pin
- J3, J5, J6, J8, J9: value Conn_01x02_Male -> Conn_01x02_Pin
- J4: value Conn_01x03_Female -> Conn_01x03_Pin
- J7: value Conn_01x06_Female -> Conn_01x06_Pin
- R1, R10, R12, R13, R7, R8, R9: value 10k - RC0805FR-0710KL -> 10K
- R11, R14: value 82 - 0805W8F820JT5E -> 1K
- R15, R16: value 10k -> 10K
- R2: value 12K 1% - 0805W8F1202T5E -> 12K 1%
- R3: renamed from R4; value 150 - 0805W8J0151T5E -> 150
- R5, R6: value 10k -> 1K
- U5, U6: value TAR5SxxU_SOT353F -> TAR5SxxU
- U8: value caravel-M.2-card -> M.2-CONNECTOR-E
- Y1: value CSTNE12M0GH5L000R0 -> 12MHz
- moved C16 45.5 mm to (159.4, 136.7), turned to 90 degrees
- moved R11 45.3 mm to (161.6, 128.8)
- moved D3 42.1 mm to (162.7, 134.4), turned to 90 degrees
- moved J8 19.0 mm to (114.0, 140.7), turned to 180 degrees
- moved C4 16.4 mm to (157.1, 136.7), turned to -90 degrees
- moved T2 16.2 mm to (133.4, 143.1)
- moved T1 16.0 mm to (133.3, 147.6)
- moved C14 13.5 mm to (113.5, 131.5), turned to 180 degrees
- moved C5 13.2 mm to (153.6, 133.3)
- moved U6 11.5 mm to (116.6, 134.4)
- moved R16 11.3 mm to (119.0, 131.3), turned to 0 degrees
- moved J5 10.5 mm to (121.9, 140.9)
- moved J9 10.5 mm to (126.4, 140.9)
- moved C6 10.5 mm to (149.3, 132.8), turned to -90 degrees
- moved C7 9.90 mm to (146.6, 132.9), turned to -90 degrees
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Connections:
- net Caravel_CSB renamed /Caravel_CSB
- net Caravel_D0 renamed /Caravel_D0
- net Caravel_D1 renamed /Caravel_D1
- net Caravel_SCK renamed /Caravel_SCK
- net FTDI_D+ renamed /FTDI_D+
- net FTDI_D- renamed /FTDI_D-
- net Net-(D2-K) renamed /ACBUS2
- net Net-(J6-Pin_1) renamed /OSC_EN
- net Net-(U1-VCCA) renamed /VCCA
- net Net-(U1-VCCCORE) renamed /VCCCORE
- net Net-(U1-~{RESET}) renamed /~{FTDI_RST}
- net Net-(U5-Noise) renamed /Noise_3V3
- net Net-(U6-Noise) renamed /Noise_1V8
- net UART_EN renamed /ACBUS0
- net USB_CS1 renamed /USB_CS1
- net USB_SCK_TXD renamed /USB_SCK_TXD
- net USB_SI renamed /USB_SI
- net USB_SO_RXD renamed /USB_SO_RXD
- net gpio renamed /gpio
- net mprj_io[0] renamed /mprj_io[0]
- net mprj_io[10] renamed /mprj_io[10]
- net mprj_io[11] renamed /mprj_io[11]
- net mprj_io[12] renamed /mprj_io[12]
- net mprj_io[13] renamed /mprj_io[13]
- net mprj_io[14] renamed /mprj_io[14]
- net mprj_io[15] renamed /mprj_io[15]
- net mprj_io[16] renamed /mprj_io[16]
- net mprj_io[17] renamed /mprj_io[17]
- net mprj_io[18] renamed /mprj_io[18]
- net mprj_io[19] renamed /mprj_io[19]
- net mprj_io[20] renamed /mprj_io[20]
- net mprj_io[21] renamed /mprj_io[21]
- net mprj_io[22] renamed /mprj_io[22]
- net mprj_io[23] renamed /mprj_io[23]
- net mprj_io[24] renamed /mprj_io[24]
- net mprj_io[25] renamed /mprj_io[25]
- net mprj_io[26] renamed /mprj_io[26]
- net mprj_io[27] renamed /mprj_io[27]
- net mprj_io[28] renamed /mprj_io[28]
- net mprj_io[29] renamed /mprj_io[29]
- net mprj_io[30] renamed /mprj_io[30]
- net mprj_io[31] renamed /mprj_io[31]
- net mprj_io[32] renamed /mprj_io[32]
- net mprj_io[33] renamed /mprj_io[33]
- net mprj_io[5]_ser_rx renamed /mprj_io[5]_ser_rx
- net mprj_io[6]_ser_tx renamed /mprj_io[6]_ser_tx
- net mprj_io[7] renamed /mprj_io[7]
- net mprj_io[8] renamed /mprj_io[8]
- net mprj_io[9] renamed /mprj_io[9]
- net vccd renamed +1V8
- net vccd2 renamed /vccd2
- net vdda1 renamed /vdda1
- net vdda2 renamed /vdda2
- net xclk renamed /xclk
- net ~{MEM_HOLD} renamed /~{MEM_HOLD}
- net ~{MEM_WP} renamed /~{MEM_WP}
- C12 pad 2: vdda -> +3V3
- C16 pad 1: GND -> +3V3
- C16 pad 2: vdda -> GND
- C17 pad 1: vdda -> GND
- C17 pad 2: GND -> +3V3
- C4 pad 2: vdda -> +3V3
- C5 pad 2: vdda -> +3V3
- C6 pad 2: vdda -> +3V3
- C7 pad 2: vdda -> +3V3
- C8 pad 2: vdda -> +3V3
- C9 pad 2: vdda -> +3V3
- J1 pad 1: +5V -> VBUS
- J10 pad 1: mprj_io[37] -> /ACBUS1
- J10 pad 2: mprj_io[36] -> GND
- J10 pad 3: mprj_io[35] -> +3V3
- J10 pad 4: mprj_io[34] -> /mprj_io[37]
- J10 pad 5: ~{RST} -> /mprj_io[36]
- J10 pad 6: GND -> /mprj_io[35]
- J10 pad 7: vdda -> /mprj_io[34]
- J11 pad 26: vdda -> +3V3
- J11 pad 27: vdda -> +3V3
- J2 pad 1: GND -> +3V3
- J4 pad 1: vdda -> +3V3
- J5 pad 1: vdda -> +3V3
- J5 pad 2: vdda -> +3V3
- J9 pad 1: vdda -> +3V3
- J9 pad 2: vdda -> +3V3
- R1 pad 2: vdda -> +3V3
- R10 pad 2: vdda -> +3V3
- R11 pad 1: vdda -> +3V3
- R12 pad 2: vdda -> +3V3
- R13 pad 2: vdda -> +3V3
- R14 pad 1: vdda -> +3V3
- R3 pad 2: vdda -> +3V3
- R5 pad 1: vdda -> GND
- R6 pad 1: vdda -> GND
- R7 pad 2: vdda -> +3V3
- R8 pad 2: vdda -> +3V3
- R9 pad 2: vdda -> +3V3
- SW1 pad 1: ~{MR} -> /ACBUS1
- U1 pad 12: vdda -> +3V3
- U1 pad 17: unconnected-(U1-ADBUS4-Pad17) -> /ADBUS4
- U1 pad 18: unconnected-(U1-ADBUS5-Pad18) -> /ADBUS5
- U1 pad 19: unconnected-(U1-ADBUS6-Pad19) -> /ADBUS6
- U1 pad 20: unconnected-(U1-ADBUS7-Pad20) -> /ADBUS7
- U1 pad 24: vdda -> +3V3
- U1 pad 25: ~{MR} -> /ACBUS1
- U1 pad 27: Net-(D1-K) -> /ACBUS3
- U1 pad 28: unconnected-(U1-ACBUS4-Pad28) -> /ACBUS4
- U1 pad 29: unconnected-(U1-ACBUS5-Pad29) -> /ACBUS5
- U1 pad 3: vdda -> +3V3
- U1 pad 30: unconnected-(U1-ACBUS6-Pad30) -> /ACBUS6
- U1 pad 31: unconnected-(U1-ACBUS7-Pad31) -> /ACBUS7
- U1 pad 39: vdda -> +3V3
- U1 pad 40: vdda -> +3V3
- U1 pad 46: vdda -> +3V3
- U1 pad 8: vdda -> +3V3
- U2 pad 5: vdda -> +3V3
- U3 pad 5: vdda -> +3V3
- U5 pad 4: vdda -> +3V3
- U7 pad 8: vdda -> +3V3
- U8 pad 16: vdda -> +3V3
- U8 pad 20: mprj_io[37] -> /mprj_io[37]
- U8 pad 22: mprj_io[36] -> /mprj_io[36]
- U8 pad 3: vdda -> +3V3
- U8 pad 32: mprj_io[35] -> /mprj_io[35]
- U8 pad 34: mprj_io[34] -> /mprj_io[34]
- U8 pad 5: vdda -> +3V3
- U8 pad 7: ~{RST} -> /ACBUS1
- X1 pad 4: vdda -> +3V3
Routing:
- net +3V3: track 0.00 -> 403.3 mm, vias 0 -> 17
- net vdda: track 379.7 -> 0.00 mm, vias 20 -> 0
- net /ACBUS1: track 0.00 -> 126.3 mm, vias 0 -> 2
- net ~{RST}: track 82.2 -> 0.00 mm, vias 3 -> 0
- net ~{MR}: track 76.8 -> 0.00 mm, vias 4 -> 0
- net mprj_io[37]: track 68.4 -> 0.00 mm
- net mprj_io[36]: track 65.8 -> 0.00 mm
- net mprj_io[35]: track 62.6 -> 0.00 mm
- net mprj_io[34]: track 60.5 -> 0.00 mm
- net /mprj_io[37]: track 0.00 -> 60.3 mm
- net /mprj_io[36]: track 0.00 -> 57.7 mm
- net /mprj_io[35]: track 0.00 -> 54.6 mm
- net /mprj_io[34]: track 0.00 -> 52.3 mm
- net +1V8: track 263.7 -> 245.2 mm, vias 10 -> 8
- net /ADBUS4: track 0.00 -> 15.6 mm
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Other:
- board text added: "ADBUS4"
- board text added: "ADBUS5"
- board text added: "ADBUS6"
- board text added: "ADBUS7"
- board text added: "OSC ~{EN}"
- board text added: "REV 5B"
- board text added: "SW1"
- board text added: "UART ~{EN}"
- board text added: "~{CS}"
- board text removed: "CS"
- board text removed: "REV 5A"
